File: PCB Design/Chassis/Chassis.kicad_sch (KiCad schematic)
At the start: 57 parts, among them J1 5V voltage regulator, J10 Conn_01x02, J11 Conn_01x02, J12 Conn_01x02, J13 Conn_01x02, J14 Voltage Regulator 12v, J15 Conn_01x02, J2 Conn_01x02, J3 Conn_01x02, J4 Conn_01x02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

Commit message: pcb progress
Parts:
- added J16: microcontroller extension header, AA_Oscars_Custom:simple 01x06, symbol Connector:Conn_01x16_Pin
- added J17: Microcontroller extension header, AA_Oscars_Custom:simple 01x12, symbol Connector:Conn_01x12_Pin
- J1: footprint (none) -> AA_Oscars_Custom:5v voltage regulator
Connections:
- net gnd: now also J16.4 (Pin_4)
- net at A1.9 (A4), R11.2: now also J16.9 (Pin_9)
- net at A1.5 (A0), R7.2: now also J16.5 (Pin_5)
- net at A1.10 (A5), R12.2: now also J16.10 (Pin_10)
- net at A1.7 (A2), R9.2: now also J16.7 (Pin_7)
- net at A1.8 (A3), R10.2: now also J16.8 (Pin_8)
- net at A1.1 (~{RESET}): now also J16.1 (Pin_1)
- net at A1.11 (SCK): now also J16.11 (Pin_11)
- net at A1.12 (MOSI): now also J16.12 (Pin_12)
- net at A1.13 (MISO): now also J16.13 (Pin_13)
- net at A1.14 (RX): now also J16.14 (Pin_14)
- net at A1.15 (TX): now also J16.15 (Pin_15)
- net at A1.2 (3V3): now also J16.2 (Pin_2)
- net at A1.3 (AREF): now also J16.3 (Pin_3)
- net at A1.6 (A1), R8.2: now also J16.6 (Pin_6)
