File: PCB Design/chassis v2 daughterboard/mosfet subsystem.kicad_sch (KiCad schematic)
At the start: 5 parts, among them CN3 microblade connector, CN4 std 2 pin 2.54mm pitch, Q2 NMOS

Commit message: stable somewhat
Parts:
- CN3: footprint custom footprints:MOLEX_53047-0210_test -> chassis v2 primary board:modified jst zh used
- Q2: footprint Package_TO_SOT_SMD:SOT-23-3 -> chassis v2 primary board:Big Mosfet Old Style
Changed lines of the file:
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@@
 			)
 		)
-		(property "Footprint" "custom footprints:MOLEX_53047-0210_test"
+		(property "Footprint" "chassis v2 primary board:modified jst zh used"
 			(at 149.86 62.23 0)
 			(effects
@@
 			)
 		)
-		(property "Footprint" "Package_TO_SOT_SMD:SOT-23-3"
+		(property "Footprint" "chassis v2 primary board:Big Mosfet Old Style"
 			(at 137.668 91.186 0)
 			(effects
